File: HW/nixie_controller.sch (EAGLE design)
At the start: 51 parts, among them IC2 LM386M-1, IC3 7812TV, J1 POWER_JACKPTH_LOCK, Q2 FDN340P, Q3 CMPT5551

Commit message: uprava sch
Parts:
- added D7: 1N4148, adafruit:DIODESOD-123
- added REL: (no value), con-wago-500:W237-103
- added SV2: (no value), con-lstb:MA04-1
- added U$3: 41.61.9.012.0010, 41.52.9.024.0010:41.61.9.012.0010
- added VYP_IN, VYP_OUT: LSP11, solpad:LSP11
Connections:
- new net N$14: J1.PWR, VYP_IN.MP
- new net N$15: VYP_OUT.MP
- new net N$21: J1.GND, J1.GNDBREAK
- new net N$30: REL-3.KL, U$3G$2.S
- new net RX: SV2.3, WEMOS1.RX
- new net TX: SV2.2, WEMOS1.TX
- net +5V: now also SV2.1
- net GND: now also SV2.4
- net N$8: now also REL-1.KL, U$3G$2.O; no longer WEMOS1.TX
- net N$9: now also REL-2.KL, U$3G$2.P; no longer WEMOS1.RX
Other:
- note removed: "MAX 3V3"
- moved on the sheet: J1
Changed lines of the file:
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@@
 <part name="GND5" library="supply1" library_urn="urn:adsk.eagle:library:371" deviceset="GND" device=""/>
 <part name="GND6" library="supply1" library_urn="urn:adsk.eagle:library:371" deviceset="GND" device=""/>
+<part name="SV2" library="con-lstb" library_urn="urn:adsk.eagle:library:162" deviceset="MA04-1" device="" package3d_urn="urn:adsk.eagle:package:8337/1"/>
+<part name="VYP_IN" library="solpad" library_urn="urn:adsk.eagle:library:364" deviceset="LSP11" device="" package3d_urn="urn:adsk.eagle:package:26502/1"/>
+<part name="VYP_OUT" library="solpad" library_urn="urn:adsk.eagle:library:364" deviceset="LSP11" device="" package3d_urn="urn:adsk.eagle:package:26502/1"/>
+<part name="GND7" library="supply1" library_urn="urn:adsk.eagle:library:371" deviceset="GND" device=""/>
+<part name="U$3" library="41.52.9.024.0010" deviceset="41.61.9.012.0010" device=""/>
+<part name="REL" library="con-wago-500" library_urn="urn:adsk.eagle:library:195" deviceset="W237-103" device="" package3d_urn="urn:adsk.eagle:package:10691/1"/>
+<part name="D7" library="adafruit" library_urn="urn:adsk.eagle:library:420" deviceset="DIODE" device="SOD-123" package3d_urn="urn:adsk.eagle:package:6240753/1" value="1N4148"/>
 </parts>
 <sheets>
@@
 <text x="181.61" y="198.882" size="1.778" layer="97">190V</text>
 <text x="114.554" y="191.008" size="1.778" layer="97">212mV</text>
-<text x="99.06" y="81.28" size="1.778" layer="91">MAX 3V3</text>
 <text x="88.9" y="30.48" size="1.778" layer="91">ochranou ZD</text>
 <text x="109.22" y="119.38" size="1.778" layer="91">
@@
 <attribute name="VALUE" x="33.02" y="167.64" size="1.778" layer="96"/>
 </instance>
-<instance part="J1" gate="G$1" x="-38.1" y="129.54" smashed="yes">
-<attribute name="VALUE" x="-48.26" y="139.7" size="1.778" layer="96" font="vector"/>
-<attribute name="NAME" x="-48.26" y="129.54" size="1.778" layer="95" font="vector"/>
+<instance part="J1" gate="G$1" x="22.86" y="358.14" smashed="yes">
+<attribute name="VALUE" x="12.7" y="368.3" size="1.778" layer="96" font="vector"/>
+<attribute name="NAME" x="12.7" y="358.14" size="1.778" layer="95" font="vector"/>
 </instance>
 <instance part="L2" gate="G$1" x="91.44" y="205.74" smashed="yes">
@@
 <instance part="GND6" gate="1" x="83.82" y="119.38" smashed="yes">
 <attribute name="VALUE" x="81.28" y="116.84" size="1.778" layer="96"/>
+</instance>
+<instance part="SV2" gate="1" x="228.6" y="43.18" smashed="yes" rot="MR0">
+<attribute name="VALUE" x="229.87" y="33.02" size="1.778" layer="96" rot="MR0"/>
+<attribute name="NAME" x="229.87" y="49.022" size="1.778" layer="95" rot="MR0"/>
+</instance>
+<instance part="VYP_IN" gate="1" x="48.26" y="365.76" smashed="yes" rot="R270">
+<attribute name="NAME" x="46.99" y="368.681" size="1.778" layer="95"/>
+</instance>
+<instance part="VYP_OUT" gate="1" x="63.5" y="365.76" smashed="yes" rot="R90">
+<attribute name="NAME" x="59.69" y="368.681" size="1.778" layer="95"/>
+</instance>
+<instance part="GND7" gate="1" x="127" y="320.04" smashed="yes">
+<attribute name="VALUE" x="124.46" y="317.5" size="1.778" layer="96"/>
+</instance>
+<instance part="U$3" gate="G$1" x="238.76" y="266.7" smashed="yes">
+<attribute name="VALUE" x="217.17" y="269.621" size="1.778" layer="96"/>
+<attribute name="PART" x="217.17" y="271.78" size="1.778" layer="95"/>
+</instance>
+<instance part="U$3" gate="G$2" x="274.32" y="266.7" smashed="yes" rot="R90">
+<attribute name="PART" x="274.32" y="269.24" size="1.778" layer="95" rot="R90"/>
+</instance>
+<instance part="REL" gate="-1" x="289.56" y="271.78" smashed="yes" rot="MR0">
+<attribute name="NAME" x="289.56" y="272.669" size="1.778" layer="95" rot="MR180"/>
+</instance>
+<instance part="REL" gate="-2" x="289.56" y="266.7" smashed="yes" rot="MR0">
+<attribute name="NAME" x="289.56" y="267.589" size="1.778" layer="95" rot="MR180"/>
+</instance>
+<instance part="REL" gate="-3" x="289.56" y="261.62" smashed="yes" rot="MR0">
+<attribute name="VALUE" x="292.1" y="257.937" size="1.778" layer="96" rot="MR0"/>
+<attribute name="NAME" x="289.56" y="262.509" size="1.778" layer="95" rot="MR180"/>
+</instance>
+<instance part="D7" gate="G$1" x="248.92" y="266.7" smashed="yes" rot="R90">
+<attribute name="NAME" x="253.746" y="265.43" size="1.27" layer="95" rot="R90"/>
+<attribute name="VALUE" x="251.968" y="263.652" size="1.27" layer="96" rot="R90"/>
 </instance>
 </instances>
@@
 <wire x1="83.82" y1="127" x2="83.82" y2="121.92" width="0.1524" layer="91"/>
 <pinref part="GND6" gate="1" pin="GND"/>
+</segment>
+<segment>
+<pinref part="SV2" gate="1" pin="4"/>
+<wire x1="220.98" y1="45.72" x2="208.28" y2="45.72" width="0.1524" layer="91"/>
+<label x="208.28" y="45.72" size="1.778" layer="95"/>
 </segment>
 </net>
@@
 <pinref part="WEMOS1" gate="D1" pin="RESET"/>
 <wire x1="121.92" y1="83.82" x2="111.76" y2="83.82" width="0.1524" layer="91"/>
-</segment>
-</net>
-<net name="N$8" class="0">
-<segment>
-<pinref part="WEMOS1" gate="D1" pin="TX"/>
-<wire x1="154.94" y1="83.82" x2="165.1" y2="83.82" width="0.1524" layer="91"/>
-</segment>
-</net>
-<net name="N$9" class="0">
-<segment>
-<pinref part="WEMOS1" gate="D1" pin="RX"/>
-<wire x1="154.94" y1="81.28" x2="165.1" y2="81.28" width="0.1524" layer="91"/>
 </segment>
 </net>
@@
 <pinref part="P+8" gate="1" pin="+5V"/>
 <wire x1="142.24" y1="254" x2="142.24" y2="251.46" width="0.1524" layer="91"/>
+</segment>
+<segment>
+<pinref part="SV2" gate="1" pin="1"/>
+<wire x1="220.98" y1="38.1" x2="208.28" y2="38.1" width="0.1524" layer="91"/>
+<label x="208.28" y="38.1" size="1.778" layer="95"/>
 </segment>
 </net>
@@
 </segment>
 </net>
+<net name="TX" class="0">
+<segment>
+<pinref part="SV2" gate="1" pin="2"/>
+<wire x1="220.98" y1="40.64" x2="208.28" y2="40.64" width="0.1524" layer="91"/>
+<label x="208.28" y="40.64" size="1.778" layer="95"/>
+</segment>
+<segment>
+<pinref part="WEMOS1" gate="D1" pin="TX"/>
+<wire x1="154.94" y1="83.82" x2="165.1" y2="83.82" width="0.1524" layer="91"/>
+<label x="157.48" y="83.82" size="1.778" layer="95"/>
+</segment>
+</net>
+<net name="RX" class="0">
+<segment>
+<pinref part="SV2" gate="1" pin="3"/>
+<wire x1="220.98" y1="43.18" x2="208.28" y2="43.18" width="0.1524" layer="91"/>
+<label x="208.28" y="43.18" size="1.778" layer="95"/>
+</segment>
+<segment>
+<pinref part="WEMOS1" gate="D1" pin="RX"/>
+<wire x1="154.94" y1="81.28" x2="165.1" y2="81.28" width="0.1524" layer="91"/>
+<label x="157.48" y="81.28" size="1.778" layer="95"/>
+</segment>
+</net>
+<net name="N$14" class="0">
+<segment>
+<pinref part="J1" gate="G$1" pin="PWR"/>
+<pinref part="VYP_IN" gate="1" pin="MP"/>
+<wire x1="25.4" y1="365.76" x2="45.72" y2="365.76" width="0.1524" layer="91"/>
+</segment>
+</net>
+<net name="N$15" class="0">
+<segment>
+<pinref part="VYP_OUT" gate="1" pin="MP"/>
+<wire x1="66.04" y1="365.76" x2="78.74" y2="365.76" width="0.1524" layer="91"/>
+</segment>
+</net>
+<net name="N$21" class="0">
+<segment>
+<pinref part="J1" gate="G$1" pin="GNDBREAK"/>
+<wire x1="25.4" y1="363.22" x2="30.48" y2="363.22" width="0.1524" layer="91"/>
+<wire x1="30.48" y1="363.22" x2="30.48" y2="360.68" width="0.1524" layer="91"/>
+<pinref part="J1" gate="G$1" pin="GND"/>
+<wire x1="25.4" y1="360.68" x2="30.48" y2="360.68" width="0.1524" layer="91"/>
+</segment>
+</net>
+<net name="N$8" class="0">
+<segment>
+<pinref part="U$3" gate="G$2" pin="O"/>
+<pinref part="REL" gate="-1" pin="KL"/>
+<wire x1="269.24" y1="271.78" x2="284.48" y2="271.78" width="0.1524" layer="91"/>
+</segment>
+</net>
+<net name="N$9" class="0">
+<segment>
+<pinref part="U$3" gate="G$2" pin="P"/>
+<pinref part="REL" gate="-2" pin="KL"/>
+<wire x1="276.86" y1="266.7" x2="284.48" y2="266.7" width="0.1524" layer="91"/>
+</segment>
+</net>
+<net name="N$30" class="0">
+<segment>
+<pinref part="U$3" gate="G$2" pin="S"/>
+<pinref part="REL" gate="-3" pin="KL"/>
+<wire x1="269.24" y1="261.62" x2="284.48" y2="261.62" width="0.1524" layer="91"/>
+</segment>
+</net>

Commit message: Update SCH+BRD
Parts:
- removed D9: FN5818, Seeed-Diode:SMD-DIODE-SCHOTTKY-40V-1A(DO-214AC)
- removed L1: VLS6045EX-101M, VLS6045EX-471M:VLS6045EX-471M
- added C13, C31, C7: 10u, rcl:C-EUC1206
- added C22, C23: 100u, Seeed-Capacitor:ALUMINUM-SMD-220UF-16V(D6.3-H7.7MM)
- added C24, C26, C27, C28, C29, C30: 100n, rcl:C-EUC1206
- added C25: 47n, rcl:C-EUC1206
- added D10: CGRM4004-G, diode:CGRM4004-G
- added D11: 1N4148, diode:CGRM4004-G
- added D12: SS33, diode:SCHOTTKY-DIODESMC
- added D8: ZD-PDZ3.6, diode:DIODE-SOD123
- added F1: MINISMDC150F/24-2, adafruit:PTCFUSE-1812
- added IC1: INA138, burr-brown:INA138
- added IC4: DG408DYTSSOP-16, maxim_sTSSOP16:DG408DYTSSOP-16
- added IC5, IC6: OPA317DBV, linear:TS931ILT
- added IC7, IC8: OPA340U, burr-brown:OPA340U
- added L3: 120R-3,5A, Seeed-Inductor:SMD-FERRITE-BEAD-470R-2A(0805)'0805'
- added L4: 7447709101, SamacSys_Parts:7447709101
- added LED1: REL_ON, led:LEDCHIP-LED0805
- added LED2: +5V_OK, led:LEDCHIP-LED0805
- added LED3: +12V_OK, led:LEDCHIP-LED0805
- added LED4: VN_ON, led:LEDCHIP-LED0805
- added Q4, Q6: CMPT5551, semicon-smd-ipc:NPN-TRANSISTOR_SOT23
- added Q5: FMMT558QTA, User-Submitted:TRANSISTOR_PNPSMD
- added Q7: MMBT3906, User-Submitted:TRANSISTOR_PNPSMD
- added R14, R27: 470R, rcl:R-EU_R1206
- added R15, R16, R18: 1k5, rcl:R-EU_R1206
- added R17: 5k1, rcl:R-EU_R1206
- added R19: 5R, rcl:R-EU_R1206
- added R20: 200k W5, rcl:R-EU_R1206
- added R21: 300k, rcl:R-EU_R1206
- added R22, R24: 15k, rcl:R-EU_R1206
- added R23, R25: 68k, rcl:R-EU_R1206
- added R26, R30, R31, R32, R33, R34: 10k, rcl:R-EU_R1206
- added R28: 220, rcl:R-EU_R1206
- added R29: 11k, rcl:R-EU_R1206
- added T1, T2: MMBT3904, DC_LOAD_AU:MMBT3904LT1-NPN-SOT23-BEC
- added TR1: SMAJ18A-TR, transil:SMAJ33CA-TR__DO214AC+MINIMELF
- added U$4: GW22LCV, 41.52.9.024.0010:GW22LCV
- added U1: (no value), SparkFun-IC-Logic:74595
- C11: value 10u -> 1u
- D5, D6: value 1N4148 -> CGRM4004-G; device adafruit:DIODESOD-123 -> diode:CGRM4004-G
- D7: value 1N4148 -> ZD-PDZ10; device adafruit:DIODESOD-123 -> diode:DIODE-SOD123
- Q2: value FDN340P -> CMPT5551; device Seeed-Transistor:SMD-MOSFET-P-CH-20V-2A-FDN340P(SOT-23) -> semicon-smd-ipc:NPN-TRANSISTOR_SOT23
- R10: value 1k -> 2k7
- R2: value 68k -> 27k
- R4: value 1k5 -> 2k2
- R5: value 47k -> 11k
- R7: value 1M/1% -> 1M
- R8: value 2k7/1% -> 4k3
- R9: value 4k3 -> 1M
Connections:
- new net +3V3: R4.2, WEMOS1.3V3
- new net MULADC: IC4.D, WEMOS1.A0
- new net N$32: LED3.A, R17.1
- new net N$33: Q4.B, R14.1
- new net N$34: LED1.A, R15.1
- new net N$35: F1.2, TR1.P$2, U$4.COM1, VYP_IN.MP
- new net N$36: IC4.EN
- new net N$37: IC4.A2
- new net N$38: IC4.A1
- new net N$39: IC4.A0
- new net N$40: LED4.A, R18.1
- new net N$41: Q6.B, R27.2
- new net N$42: C26.2, D7.A, IC1.V-, Q5.B, R20.1
- new net N$43: IC1.OUT, Q5.E
- new net N$45: C31.1, IC8.-IN, R31.1, R32.2
- new net N$46: R28.1, T1.C
- new net N$47: Q7.E, T1.B, T2.B, T2.C
- new net N$48: IC7.+IN, IC8.OUT, R31.2
- new net N$49: IC8.+IN, R33.1, R34.2
- new net N$50: Q7.B, R30.2
- new net N$51: IC7.OUT, R30.1
- new net N$52: IC7.-IN, Q7.C, R29.1
- new net OV_OC: Q2.C, Q3.C
- new net REL_ON: R14.2, R15.2
- new net VN_CTRL: R32.1
- new net VN_I: IC5.-IN, IC5.OUT
- new net VN_I_SENSE: C25.1, IC5.+IN, Q5.C, R21.1, R23.1
- new net VN_NIXIE_SHUNT: C16.1, C19.+, C26.1, D3.C, D7.C, IC1.IN-, IC1.V+, R19.2, R7.2, R9.2
- new net VN_ON: R18.2
- new net VN_U: IC6.-IN, IC6.OUT
- new net VN_U_SENSE: IC6.+IN, R10.2, R25.1, R9.1
- net +12V: now also D10.A, D5.C, IC4.V+, R17.2, U$3G$1.1; no longer D5.A
- net +5V: now also C27.1, C28.1, C29.1, C30.1, C7.1, IC5.V+, IC6.V+, IC7.V+, IC8.V+, L4.2, R16.2, R26.1, R29.2, R34.1; no longer L1.2, R4.2
- net GND: now also C13.2, C22.-, C23.-, C24.2, C25.2, C27.2, C28.2, C29.2, C30.2, C31.2, C7.2, D12.A, D5.A, D8.A, IC2.-IN, IC4.GND, IC4.V-, IC5.V-, IC6.V-, IC7.V-, IC8.V-, J1.GND, J1.GNDBREAK, LED1.C, LED2.C, LED3.C, LED4.C, Q2.E, Q4.E, Q6.E, R10.1, R20.2, R21.2, R22.2, R24.2, R33.2, T1.E, T2.E, TR1.P$1; no longer D6.A, D9.+
- net N$14: now also F1.1; no longer VYP_IN.MP
- net N$15: now also L3.1, U$4.NO1
- net N$19: now also LED2.A, R16.1; no longer C12.1, C14.1, L2.1, Q2.D, R6.1, U$1.VIN
- net N$20: no longer IC2.-IN
- net N$21: now also D11.A, Q6.C, R26.2; no longer J1.GND, J1.GNDBREAK
- net N$26: now also D11.C, R28.2
- net N$27: now also Q2.B, R22.1, R23.2; no longer Q2.G, Q3.C, R10.2
- net N$29: now also R24.1, R25.2; no longer R9.2
- net N$3: now also D12.C, L4.1; no longer D9.-, L1.1
- net N$7: now also D6.A, Q4.C, U$3G$1.2; no longer WEMOS1.3V3
- net NOISE_AD: now also D8.C; no longer WEMOS1.A0
- net UCC: now also C12.1, C13.1, C14.1, C22.+, C23.+, C24.1, D10.C, L2.1, L3.2, R6.1, U$1.VIN; no longer D5.C, Q2.S, R10.1
- net VN_EN: now also R27.1; no longer R9.1
- net VN_NIXIE: now also IC1.IN+, R19.1; no longer C16.1, C19.+, D3.C, R7.2
Other:
- note added: "1812 Udržovací 1,5A 24V vypínací 3A"
- note added: "GW22LCV"
- note added: "VN"
- note added: "ZD PCT"
- note added: "cca. 50-250V"
- note added: "dodělat: vstupy výstupy měření I, nastavování VN, monitoring U,"
- note removed: "190V"
- note removed: "ochranou ZD"

Commit message: Pokrok ve schematu
Parts:
- added C32: 100n, rcl:C-EUC1206
- added C33: 1u5, rcl:C-EUC1206
- added D13, D9: CGRM4004-G, diode:CGRM4004-G
- added D14: ZD-PDZ3.3, diode:DIODE-SOD123
- added H1, H2, H3, H4, H5, H6: MOUNT-HOLE3.0, holes:MOUNT-HOLE3.0
- added IC9: NE555D, adafruit:NE555D
- added LED5: STASTUS_1, led:LEDCHIP-LED0805
- added LS1: CEM-1201(42), CEM-1201_42_:CEM-1201(42)
- added Q8, Q9: CMPT5551, semicon-smd-ipc:NPN-TRANSISTOR_SOT23
- added R35, R36, R37, R52: 1k, rcl:R-EU_R1206
- added R38, R39, R40, R42, R46, R47, R49, R50, R51: 10k, rcl:R-EU_R1206
- added R41: 1k5, rcl:R-EU_R1206
- added R43: 4k7, rcl:R-EU_R1206
- added R44, R45: 470R, rcl:R-EU_R1206
- added R48: 20k, rcl:R-EU_R1206
- added U$5, U$6: KSC421, 41.52.9.024.0010:KSC421
- added U$7: LIGT_CONDUCT_5LED, 41.52.9.024.0010:LIGT_CONDUCT_5LED
- added U2: (no value), SparkFun-IC-Logic:74595
- R10: value 2k7 -> 8k2
- R15, R18: value 1k5 -> 680R
- R26: value 10k -> 100k
- R5: value 11k -> 10k
Connections:
- net N$37 renamed MUL_A2
- net N$38 renamed MUL_A1
- net N$39 renamed MUL_A0
- removed net OE: SV1.3
- removed net VN_ON: R18.2
- new net BTN_1: IC4.S6, R39.2, U$5.P
- new net BTN_2: IC4.S7, R40.2, U$6.P
- new net BUZZER_ON: R37.2
- new net LED_BR: R44.1
- new net LED_TR: R45.1
- new net N$37: U1.QA
- new net N$38: U1.QB
- new net N$39: U1.QC
- new net N$44: C32.1, IC9.CV
- new net N$53: C33.1, D9.C, IC9.THR, IC9.TR, R35.2
- new net N$54: D9.A, IC9.DIS, R35.1, R36.1
- new net N$55: D13.C, IC9.Q, LS1.P
- new net N$56: LED5.A, R41.1
- new net N$57: IC9.V+, Q8.E, R36.2
- new net N$58: Q8.B, R37.1
- new net N$59: D11.A, Q6.C, R26.2, R43.1
- new net N$60: Q9.B, R46.2
- new net N$61: R42.1, U$4.COM
- new net N$62: U1.QD
- new net N$63: U1.QE
- new net N$64: U1.QF
- new net N$65: U1.QG
- new net N$66: U1.QH
- new net N$67: U2.QA
- new net N$68: U2.QB
- new net N$69: U2.QC
- new net N$70: U2.QD
- new net N$71: U2.QE
- new net N$72: U2.QF
- new net N$73: U2.QG
- new net N$74: U2.QH
- new net PWR_STATUS: D14.C, IC4.S5, U$4.NO
- new net RCK_EIO: U1.RCK, U2.RCK
- new net RX_IN: R49.2, SV2.3
- new net SCK_EIO: U1.SCK, U2.SCK
- new net SER_EIO: U1.SER
- new net STATUS_1: R41.2
- new net TX_IN: Q9.C, R47.2, SV2.2
- new net UCC_U: IC4.S8, R51.1, R52.2
- net +12V: now also IC4.EN, IC9.R, Q8.C
- net +3V3: now also R46.1, R50.1, U$5.S, U$6.S, U1.VCC, U2.VCC
- net +5V: now also R47.1; no longer R26.1
- net GND: now also C32.2, C33.2, D13.A, D14.A, IC9.GND, LED5.C, LS1.M, R38.2, R39.1, R40.1, R43.2, R48.2, R52.1, SV1.3, U$5.GND, U$6.GND, U1.G, U1.GND, U2.G, U2.GND
- net LED_B: now also R45.2
- net LED_T: now also R44.2
- net N$21: now also U1.QH*, U2.SER; no longer D11.A, Q6.C, R26.2
- net N$33: now also R38.1
- net N$35: now also R42.2
- net N$36: now also U1.SCL, U2.SCL; no longer IC4.EN
- net NOISE_AD: now also IC4.S4
- net OV_OC: now also IC4.S3, R50.2
- net RX: now also R48.1, R49.1; no longer SV2.3
- net TX: now also Q9.E; no longer SV2.2
- net UCC: now also R26.1, R51.2
- net VN_EN: now also R18.2
- net VN_I: now also IC4.S2
- net VN_U: now also IC4.S1
Other:
- note added: "3V3 regulátor 0,5A"
- note added: "blokovací C"
- note added: "rozdělit země"
- note removed: "cca. 50-250V"
- note removed: "dodělat: vstupy výstupy měření I, nastavování VN, monitoring U,"

Commit message: Postupný postup, SCHEME DON, BRD ALMOST
Parts:
- removed C2: 100n, rcl:C-EUC1206
- removed D11: 1N4148, diode:CGRM4004-G
- removed D14: ZD-PDZ3.3, diode:DIODE-SOD123
- removed D8: ZD-PDZ3.6, diode:DIODE-SOD123
- removed R35: 1k, rcl:R-EU_R1206
- removed SV2: (no value), con-lstb:MA04-1
- removed U1, U2: (no value), SparkFun-IC-Logic:74595
- added C34, C46: 10u, rcl:C-EUC1206
- added C35, C36, C37, C38, C41, C42, C43, C44, C45: 100n, rcl:C-EUC1206
- added C39, C40: 10n, rcl:C-EUC1206
- added D15: PDZ15BGWX, adafruit:DIODESOD-123
- added D16: PDZ3.3BGWX, adafruit:DIODESOD-123
- added IC10: LD1117S33TR, SamacSys_Parts:LD1117S33TR
- added IC11: 74HC595D, 74xx-eu:74HC595D
- added JP1: (no value), pinhead:PINHD-1X3/90
- added JP2: (no value), pinhead:PINHD-1X4/90
- added Q10: DMP3099L-7, User-Submitted:MOSFET-PCHANNEL
- added Q11: MMBT3906, User-Submitted:TRANSISTOR_PNPSMD
- added R53, R54: 1k, rcl:R-EU_R1206
- added R55: 8k2, rcl:R-EU_R1206
- added R56, R57: 0R, rcl:R-EU_R1206
- added R58, R59, R60, R61, R62: 10k, rcl:R-EU_R1206
- added TP1, TP10, TP11, TP12, TP13, TP14, TP15, TP16, TP17, TP18, TP19, TP2, TP20, TP21, TP22, TP23, TP3, TP4, TP5, TP6, TP7, TP8, TP9: TPB1,27, testpad:TPB1,27
- added TR2, TR4: SMAJ5, transil:SMAJ33CA-TR__DO214AC+MINIMELF
- added TR3: SMAJ12, transil:SMAJ33CA-TR__DO214AC+MINIMELF
- D10: value CGRM4004-G -> PDZ3.3BGWX; device diode:CGRM4004-G -> adafruit:DIODESOD-123
- D5: value CGRM4004-G -> 1N4148; device diode:CGRM4004-G -> adafruit:DIODESOD-123
- R14: value 470R -> 1k
Connections:
- removed net N$21: U1.QH*, U2.SER
- removed net N$26: D11.C, R28.2, R7.1, R8.2, U$1.FB
- removed net N$36: U1.SCL, U2.SCL
- removed net N$37: U1.QA
- removed net N$62: U1.QD
- removed net N$64: U1.QF
- removed net N$65: U1.QG
- removed net N$66: U1.QH
- removed net N$67: U2.QA
- removed net N$68: U2.QB
- removed net N$69: U2.QC
- removed net N$70: U2.QD
- removed net N$71: U2.QE
- removed net N$72: U2.QF
- removed net N$73: U2.QG
- removed net N$74: U2.QH
- new net AGND: C10.2, C25.2, C9.2, D10.A, IC2.-IN, Q1.1, R21.2, R5.1, R57.2, R8.1, T1.E, T2.E
- new net EXT_MCU: JP1.2, WEMOS1.D0
- new net SW_FB: D5.C, R28.2, R7.1, R8.2, TP14.TP, U$1.FB
- net +12V: now also C36.2, C38.1, C42.1, D9.C, IC9.V+, Q11.E, R59.2, TP3.TP, TR3.P$2; no longer C2.1, D10.A, D5.C, IC9.R, Q8.C
- net +3V3: now also C34.1, C35.1, C45.1, IC10.VOUT, IC11A.SCL, IC11P.VCC, R53.2, R54.2, TP4.TP, TR2.P$2; no longer U$5.S, U$6.S, U1.VCC, U2.VCC, WEMOS1.3V3
- net +5V: now also C37.1, C41.2, C43.1, C44.1, C46.1, IC10.VIN, JP1.3, JP2.1, R56.1, TP2.TP, TR4.P$2; no longer C20.+, C7.1, L4.2, R12.1, SV2.1
- net BTN_1: now also C39.1
- net BTN_2: now also C40.1
- net BUZZER_ON: now also IC11A.QA
- net GND: now also C34.2, C35.2, C36.1, C37.2, C38.2, C39.2, C40.2, C41.1, C42.2, C43.2, C44.2, C45.2, C46.2, D16.A, IC10.GND, IC10.TAB, IC11A.G, IC11P.GND, JP1.1, JP2.4, Q8.E, R57.1, R60.1, R61.1, R62.1, TP5.TP, TR2.P$1, TR3.P$1, TR4.P$1; no longer C10.2, C2.2, C25.2, C9.2, D14.A, D5.A, D8.A, IC2.-IN, Q1.1, R21.2, R5.1, R8.1, SV2.4, T1.E, T2.E, U1.G, U1.GND, U2.G, U2.GND
- net LED_B: no longer WEMOS1.D1
- net LED_BR: now also IC11A.QE
- net LED_T: no longer WEMOS1.D0
- net LED_TR: now also IC11A.QD
- net MUL_A0: now also IC11A.QF
- net MUL_A1: now also IC11A.QG
- net MUL_A2: now also IC11A.QH
- net N$2: now also C33.1, IC9.THR, IC9.TR, R36.1, TP23.TP; no longer WEMOS1.RESET
- net N$33: now also TP20.TP
- net N$35: now also Q10.D; no longer F1.2
- net N$38: now also C20.+, C7.1, L4.2, R12.1, R56.2; no longer U1.QB
- net N$39: now also IC9.R, Q11.C, R60.2; no longer U1.QC
- net N$4: now also R53.1, U$5.S; no longer WEMOS1.D6
- net N$41: now also TP13.TP
- net N$42: now also TP11.TP
- net N$45: now also TP19.TP
- net N$47: now also TP18.TP
- net N$48: now also TP15.TP
- net N$5: now also R54.1, U$6.S; no longer WEMOS1.D7
- net N$50: now also TP16.TP
- net N$52: now also TP17.TP
- net N$53: now also Q11.B, R58.2; no longer C33.1, D9.C, IC9.THR, IC9.TR, R35.2
- net N$54: now also D13.C, IC9.Q, LS1.P, R36.2, TP22.TP; no longer IC9.DIS, R35.1, R36.1
- net N$55: now also Q8.C, R58.1, R59.1; no longer D13.C, IC9.Q, LS1.P
- net N$57: now also Q8.B, R37.1, R61.2; no longer IC9.V+, Q8.E, R36.2
- net N$58: now also D15.C, F1.2, Q10.S; no longer Q8.B, R37.1
- net N$59: now also D5.A; no longer D11.A
- net N$6: now also IC6.-IN, R55.2; no longer WEMOS1.D8
- net N$63: now also D15.A, Q10.G, R62.2; no longer U1.QE
- net NOISE_AD: now also D10.C, TP21.TP; no longer D8.C
- net PWR_STATUS: now also D16.C; no longer D14.C
- net RCK_EIO: now also IC11A.RCK, WEMOS1.D8; no longer U1.RCK, U2.RCK
- net REL_ON: now also IC11A.QB
- net RX_IN: now also JP2.3; no longer SV2.3
- net SCK_EIO: now also IC11A.SCK, WEMOS1.D7; no longer U1.SCK, U2.SCK
- net SER_EIO: now also IC11A.SER, WEMOS1.D1; no longer U1.SER
- net STATUS_1: now also IC11A.QC
- net TX_IN: now also JP2.2; no longer SV2.2
- net UCC: now also TP1.TP; no longer D10.C
- net VN_CTRL: now also WEMOS1.D6
- net VN_I: now also TP12.TP
- net VN_I_SENSE: now also TP10.TP
- net VN_NIXIE: now also TP7.TP
- net VN_NIXIE_SHUNT: now also TP6.TP
- net VN_U: now also R55.1, TP9.TP; no longer IC6.-IN
- net VN_U_SENSE: now also TP8.TP
Other:
- note removed: "3V3 regulátor 0,5A"
- note removed: "ZD PCT"
- note removed: "blokovací C"
- note removed: "rozdělit země"

Commit message: Aktualizace aktuální verze desky , nákup a pod.
Parts:
- removed H3: MOUNT-HOLE3.0, holes:MOUNT-HOLE3.0
Connections:
- net EXT_MCU: now also JP1.1; no longer JP1.2
- net GND: now also JP1.2; no longer JP1.1
